File: boards/MainCircuitSchematic.brd (EAGLE design)
At the start: 76.2 x 46.7 mm, 13 parts

Commit message: Add files via upload
fixed receiver and servo pins
Parts:
- moved RECEIVNOTHING 17.8 mm to (97.8, 57.1)
- moved RECEIVPWR 17.8 mm to (97.8, 59.7)
- moved RECIEVGND 17.8 mm to (97.8, 62.2)
- moved SERVO1 2.62 mm to (109.9, 62.2), turned to 0 degrees
- moved SERVO2 2.54 mm to (109.9, 56.5), turned to 0 degrees
Connections:
- net 7.4V: now also SERVO1.2, SERVO2.2; no longer SERVO1.3, SERVO2.3
- net N$7: now also SERVO2.3; no longer SERVO2.2
- net N$8: now also SERVO1.3; no longer SERVO1.2
Routing:
- net 5V: track 76.1 -> 55.8 mm, vias 1 -> 0
- net N$7: track 9.88 -> 16.1 mm
- net 7.4V: track 72.7 -> 77.1 mm
- net N$8: track 21.1 -> 22.7 mm
Changed lines of the file:
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@@
 <text x="77.47" y="27.94" size="1.27" layer="25">-</text>
 <text x="73.66" y="44.45" size="1.27" layer="25">-</text>
-<text x="77.47" y="62.865" size="1.27" layer="25">-</text>
-<text x="111.125" y="62.865" size="1.27" layer="25">-</text>
-<text x="111.125" y="56.515" size="1.27" layer="25">-</text>
+<text x="105.41" y="62.865" size="1.27" layer="25">-</text>
+<text x="105.41" y="57.15" size="1.27" layer="25">-</text>
 <text x="114.935" y="22.86" size="1.27" layer="25">-</text>
 <text x="121.92" y="43.18" size="1.27" layer="25">-</text>
@@
 <attribute name="VALUE" x="81.28" y="53.975" size="1.27" layer="27"/>
 </element>
-<element name="SERVO1" library="adafruit" library_urn="urn:adsk.eagle:library:420" package="1X03-CLEANBIG" package3d_urn="urn:adsk.eagle:package:6240706/1" value="" x="107.315" y="62.865" smashed="yes" rot="R180">
-<attribute name="NAME" x="111.2012" y="61.0362" size="1.27" layer="25" ratio="10" rot="R180"/>
-<attribute name="VALUE" x="111.125" y="66.04" size="1.27" layer="27" rot="R180"/>
-</element>
-<element name="SERVO2" library="adafruit" library_urn="urn:adsk.eagle:library:420" package="1X03-CLEANBIG" package3d_urn="urn:adsk.eagle:package:6240706/1" value="" x="107.315" y="56.515" smashed="yes" rot="R180">
-<attribute name="NAME" x="111.2012" y="54.6862" size="1.27" layer="25" ratio="10" rot="R180"/>
-<attribute name="VALUE" x="111.125" y="59.69" size="1.27" layer="27" rot="R180"/>
+<element name="SERVO1" library="adafruit" library_urn="urn:adsk.eagle:library:420" package="1X03-CLEANBIG" package3d_urn="urn:adsk.eagle:package:6240706/1" value="" x="109.855" y="62.23" smashed="yes">
+<attribute name="NAME" x="105.3338" y="64.0588" size="1.27" layer="25" ratio="10"/>
+<attribute name="VALUE" x="106.045" y="59.055" size="1.27" layer="27"/>
+</element>
+<element name="SERVO2" library="adafruit" library_urn="urn:adsk.eagle:library:420" package="1X03-CLEANBIG" package3d_urn="urn:adsk.eagle:package:6240706/1" value="" x="109.855" y="56.515" smashed="yes">
+<attribute name="NAME" x="105.9688" y="58.3438" size="1.27" layer="25" ratio="10"/>
+<attribute name="VALUE" x="106.045" y="53.34" size="1.27" layer="27"/>
 </element>
 <element name="BATTERY" library="Connector" library_urn="urn:adsk.eagle:library:16378166" package="1X02" package3d_urn="urn:adsk.eagle:package:22435/2" value="PINHD-1X2" x="72.39" y="41.91" smashed="yes" rot="R270">
@@
 <attribute name="TYPE" value="" x="88.9" y="60.96" size="1.778" layer="27" display="off"/>
 </element>
-<element name="RECIEVGND" library="pinhead" library_urn="urn:adsk.eagle:library:325" package="1X01" package3d_urn="urn:adsk.eagle:package:22485/2" value="" x="80.01" y="62.23" smashed="yes">
-<attribute name="POPULARITY" value="64" x="80.01" y="62.23" size="1.778" layer="27" display="off"/>
-<attribute name="VALUE" x="78.74" y="59.055" size="1.27" layer="27"/>
-</element>
-<element name="RECEIVNOTHING" library="pinhead" library_urn="urn:adsk.eagle:library:325" package="1X01" package3d_urn="urn:adsk.eagle:package:22485/2" value="" x="80.01" y="57.15" smashed="yes">
-<attribute name="POPULARITY" value="64" x="80.01" y="57.15" size="1.778" layer="27" display="off"/>
-<attribute name="VALUE" x="78.74" y="53.975" size="1.27" layer="27"/>
-</element>
-<element name="RECEIVPWR" library="pinhead" library_urn="urn:adsk.eagle:library:325" package="1X01" package3d_urn="urn:adsk.eagle:package:22485/2" value="" x="80.01" y="59.69" smashed="yes">
-<attribute name="POPULARITY" value="64" x="80.01" y="59.69" size="1.778" layer="27" display="off"/>
-<attribute name="VALUE" x="78.74" y="56.515" size="1.27" layer="27"/>
+<element name="RECIEVGND" library="pinhead" library_urn="urn:adsk.eagle:library:325" package="1X01" package3d_urn="urn:adsk.eagle:package:22485/2" value="" x="97.79" y="62.23" smashed="yes">
+<attribute name="POPULARITY" value="64" x="97.79" y="62.23" size="1.778" layer="27" display="off"/>
+<attribute name="VALUE" x="96.52" y="59.055" size="1.27" layer="27"/>
+</element>
+<element name="RECEIVNOTHING" library="pinhead" library_urn="urn:adsk.eagle:library:325" package="1X01" package3d_urn="urn:adsk.eagle:package:22485/2" value="" x="97.79" y="57.15" smashed="yes">
+<attribute name="POPULARITY" value="64" x="97.79" y="57.15" size="1.778" layer="27" display="off"/>
+<attribute name="VALUE" x="96.52" y="53.975" size="1.27" layer="27"/>
+</element>
+<element name="RECEIVPWR" library="pinhead" library_urn="urn:adsk.eagle:library:325" package="1X01" package3d_urn="urn:adsk.eagle:package:22485/2" value="" x="97.79" y="59.69" smashed="yes">
+<attribute name="POPULARITY" value="64" x="97.79" y="59.69" size="1.778" layer="27" display="off"/>
+<attribute name="VALUE" x="96.52" y="56.515" size="1.27" layer="27"/>
 </element>
 </elements>
@@
 <signal name="7.4V">
 <contactref element="BATTERY" pad="2"/>
-<contactref element="SERVO2" pad="3"/>
-<contactref element="SERVO1" pad="3"/>
 <contactref element="V-REG" pad="2"/>
 <wire x1="73.66" y1="40.64" x2="72.39" y2="40.64" width="0.6096" layer="1"/>
@@
 <wire x1="72.39" y1="29.21" x2="72.39" y2="40.64" width="0.6096" layer="1"/>
 <wire x1="76.835" y1="24.765" x2="72.39" y2="29.21" width="0.6096" layer="1"/>
-<wire x1="76.2" y1="50.8" x2="77.47" y2="52.07" width="0.6096" layer="1"/>
 <wire x1="76.2" y1="41.91" x2="74.93" y2="40.64" width="0.6096" layer="1"/>
 <wire x1="74.93" y1="40.64" x2="72.39" y2="40.64" width="0.6096" layer="1"/>
 <wire x1="76.2" y1="50.8" x2="76.2" y2="41.91" width="0.6096" layer="1"/>
-<wire x1="100.33" y1="52.07" x2="104.14" y2="55.88" width="0.6096" layer="1"/>
-<wire x1="77.47" y1="52.07" x2="100.33" y2="52.07" width="0.6096" layer="1"/>
-<wire x1="104.775" y1="62.865" x2="104.775" y2="56.515" width="0.6096" layer="1"/>
-<wire x1="104.775" y1="56.515" x2="104.14" y2="55.88" width="0.6096" layer="1"/>
+<contactref element="SERVO2" pad="2"/>
+<contactref element="SERVO1" pad="2"/>
+<wire x1="109.855" y1="62.23" x2="109.855" y2="56.515" width="0.6096" layer="1"/>
+<wire x1="109.855" y1="56.515" x2="107.95" y2="54.61" width="0.6096" layer="1"/>
+<wire x1="80.01" y1="54.61" x2="76.2" y2="50.8" width="0.6096" layer="1"/>
+<wire x1="107.95" y1="54.61" x2="80.01" y2="54.61" width="0.6096" layer="1"/>
 </signal>
 <signal name="5V">
@@
 <wire x1="113.03" y1="27.305" x2="113.03" y2="34.29" width="0.6096" layer="1"/>
 <contactref element="RECEIVPWR" pad="1"/>
-<wire x1="120.65" y1="48.26" x2="116.84" y2="52.07" width="0.6096" layer="16"/>
-<wire x1="116.84" y1="52.07" x2="101.6" y2="52.07" width="0.6096" layer="16"/>
-<wire x1="101.6" y1="52.07" x2="99.06" y2="54.61" width="0.6096" layer="16"/>
-<via x="99.06" y="54.61" extent="1-16" drill="0.35"/>
-<wire x1="99.06" y1="54.61" x2="78.74" y2="54.61" width="0.6096" layer="1"/>
-<wire x1="78.74" y1="54.61" x2="77.47" y2="55.88" width="0.6096" layer="1"/>
-<wire x1="77.47" y1="55.88" x2="77.47" y2="58.42" width="0.6096" layer="1"/>
-<wire x1="77.47" y1="58.42" x2="78.74" y2="59.69" width="0.6096" layer="1"/>
-<wire x1="78.74" y1="59.69" x2="80.01" y2="59.69" width="0.6096" layer="1"/>
+<wire x1="120.65" y1="48.26" x2="120.65" y2="55.245" width="0.6096" layer="16"/>
+<wire x1="120.65" y1="55.245" x2="116.205" y2="59.69" width="0.6096" layer="16"/>
+<wire x1="116.205" y1="59.69" x2="97.79" y2="59.69" width="0.6096" layer="16"/>
 </signal>
 <signal name="SCL_5V">
@@
 </signal>
 <signal name="N$7">
-<contactref element="SERVO2" pad="2"/>
+<contactref element="SERVO2" pad="3"/>
 <contactref element="B1" pad="4"/>
-<wire x1="107.315" y1="56.515" x2="100.33" y2="49.53" width="0.4064" layer="1"/>
+<wire x1="112.395" y1="56.515" x2="108.585" y2="52.705" width="0.4064" layer="1"/>
+<wire x1="108.585" y1="52.705" x2="101.6" y2="52.705" width="0.4064" layer="1"/>
+<wire x1="101.6" y1="52.705" x2="100.33" y2="51.435" width="0.4064" layer="1"/>
+<wire x1="100.33" y1="51.435" x2="100.33" y2="49.53" width="0.4064" layer="1"/>
 </signal>
 <signal name="N$8">
-<contactref element="SERVO1" pad="2"/>
+<contactref element="SERVO1" pad="3"/>
 <contactref element="B1" pad="3"/>
-<wire x1="107.315" y1="62.865" x2="111.76" y2="58.42" width="0.4064" layer="1"/>
-<wire x1="111.76" y1="58.42" x2="111.76" y2="54.61" width="0.4064" layer="1"/>
-<wire x1="111.76" y1="54.61" x2="110.49" y2="53.34" width="0.4064" layer="1"/>
-<wire x1="110.49" y1="53.34" x2="106.68" y2="53.34" width="0.4064" layer="1"/>
-<wire x1="106.68" y1="53.34" x2="102.87" y2="49.53" width="0.4064" layer="1"/>
+<wire x1="112.395" y1="62.23" x2="114.3" y2="60.325" width="0.4064" layer="1"/>
+<wire x1="114.3" y1="60.325" x2="114.3" y2="54.61" width="0.4064" layer="1"/>
+<wire x1="103.505" y1="51.435" x2="102.87" y2="50.8" width="0.4064" layer="1"/>
+<wire x1="102.87" y1="50.8" x2="102.87" y2="49.53" width="0.4064" layer="1"/>
+<wire x1="114.3" y1="54.61" x2="111.125" y2="51.435" width="0.4064" layer="1"/>
+<wire x1="111.125" y1="51.435" x2="103.505" y2="51.435" width="0.4064" layer="1"/>
 </signal>
 </signals>
